File: eagle/board.brd (EAGLE design)
At the start: 75 x 50 mm, 27 parts, among them SW1 C&K L202XXYYXMS, X1 2.1MMJACKTHM, X10 10p-2.0, X2 2p-2.0, X3 5p-2.54, X4 8p-2.54, X5 14p-2.54, X6 14p-2.54, X7 5p-2.54, X8 8p-2.54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

Commit message: fix silkscreen for pin 4
Parts:
- moved D1 0.25 mm to (30.7, 39.4)
- moved F1 0.25 mm to (34.7, 39.1)
- moved X2 0.13 mm to (33.7, 45.6)
Other:
- board text added: "D4"
- board text removed: "D6"
Changed lines of the file:
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@@
 <layer number="19" name="Unrouted" color="6" fill="1" visible="yes" active="yes"/>
 <layer number="20" name="Dimension" color="15" fill="1" visible="yes" active="yes"/>
-<layer number="21" name="tPlace" color="7" fill="1" visible="no" active="yes"/>
+<layer number="21" name="tPlace" color="7" fill="1" visible="yes" active="yes"/>
 <layer number="22" name="bPlace" color="7" fill="1" visible="yes" active="yes"/>
 <layer number="23" name="tOrigins" color="15" fill="1" visible="yes" active="yes"/>
@@
 <text x="53.213" y="3.81" size="1.016" layer="22" font="vector" ratio="10" rot="SMR90" align="center-right">D12</text>
 <text x="50.673" y="3.81" size="1.016" layer="22" font="vector" ratio="10" rot="SMR90" align="center-right">D11</text>
-<text x="48.133" y="3.81" size="1.016" layer="22" font="vector" ratio="10" rot="SMR90" align="center-right">D6</text>
+<text x="48.133" y="3.81" size="1.016" layer="22" font="vector" ratio="10" rot="SMR90" align="center-right">D4</text>
 <text x="48.133" y="3.81" size="1.016" layer="21" font="vector" ratio="10" rot="SR270" align="center-left">CS</text>
 <text x="50.673" y="3.81" size="1.016" layer="21" font="vector" ratio="10" rot="SR270" align="center-left">MOSI</text>
@@
 </element>
 <element name="U$1" library="thewknd" package="DCBARREL_DESC" value="" x="33.02" y="35.179"/>
-<element name="X2" library="Seeed-OPL-Connector" package="H2-2.0-6X4.5MM" value="2p-2.0" x="33.655" y="45.466" smashed="yes" rot="R180">
-<attribute name="NAME" x="37.211" y="44.704" size="1.016" layer="25" font="vector" ratio="10" rot="SR270"/>
-<attribute name="VALUE" x="36.195" y="46.736" size="0.889" layer="27" ratio="11" rot="R180"/>
-<attribute name="NAME" x="33.02" y="45.339" size="0.254" layer="33" ratio="10"/>
-</element>
-<element name="D1" library="Seeed-OPL-Diode" package="SOD-123" value="20V-1A" x="30.734" y="39.624" smashed="yes" rot="R270">
-<attribute name="MPN" value="B5819W" x="64.389" y="45.847" size="1.016" layer="27" ratio="10" rot="R270" display="off"/>
-<attribute name="NAME" x="31.877" y="41.529" size="1.016" layer="25" font="vector" ratio="10" rot="SR270"/>
-<attribute name="VALUE" x="28.702" y="41.529" size="0.889" layer="27" font="vector" ratio="11" rot="R270"/>
-<attribute name="NAME" x="30.099" y="40.513" size="0.381" layer="33" ratio="10" rot="R270"/>
+<element name="X2" library="Seeed-OPL-Connector" package="H2-2.0-6X4.5MM" value="2p-2.0" x="33.655" y="45.593" smashed="yes" rot="R180">
+<attribute name="NAME" x="37.211" y="44.831" size="1.016" layer="25" font="vector" ratio="10" rot="SR270"/>
+<attribute name="VALUE" x="36.195" y="46.863" size="0.889" layer="27" ratio="11" rot="R180"/>
+<attribute name="NAME" x="33.02" y="45.466" size="0.254" layer="33" ratio="10"/>
+</element>
+<element name="D1" library="Seeed-OPL-Diode" package="SOD-123" value="20V-1A" x="30.734" y="39.37" smashed="yes" rot="R270">
+<attribute name="MPN" value="B5819W" x="64.389" y="45.593" size="1.016" layer="27" ratio="10" rot="R270" display="off"/>
+<attribute name="NAME" x="31.877" y="41.275" size="1.016" layer="25" font="vector" ratio="10" rot="SR270"/>
+<attribute name="VALUE" x="28.702" y="41.275" size="0.889" layer="27" font="vector" ratio="11" rot="R270"/>
+<attribute name="NAME" x="30.099" y="40.259" size="0.381" layer="33" ratio="10" rot="R270"/>
 </element>
 <element name="X1" library="adafruit" package="PJ-102A" value="2.1MMJACKTHM" x="44.323" y="45.72" smashed="yes">
 <attribute name="NAME" x="49.149" y="48.768" size="1.016" layer="25" font="vector" ratio="10" rot="SR270"/>
 </element>
-<element name="F1" library="Seeed-OPL-fuse" package="F1206" value="6V/500mA" x="34.671" y="39.37" smashed="yes" rot="R270">
-<attribute name="MPN" value="SMD1206R500SF" x="62.992" y="72.263" size="1.016" layer="27" ratio="10" rot="R270" display="off"/>
-<attribute name="NAME" x="36.195" y="41.529" size="1.016" layer="25" font="vector" ratio="10" rot="SR270"/>
-<attribute name="VALUE" x="31.877" y="41.91" size="0.889" layer="27" ratio="11" rot="R270"/>
+<element name="F1" library="Seeed-OPL-fuse" package="F1206" value="6V/500mA" x="34.671" y="39.116" smashed="yes" rot="R270">
+<attribute name="MPN" value="SMD1206R500SF" x="62.992" y="72.009" size="1.016" layer="27" ratio="10" rot="R270" display="off"/>
+<attribute name="NAME" x="36.195" y="41.275" size="1.016" layer="25" font="vector" ratio="10" rot="SR270"/>
+<attribute name="VALUE" x="31.877" y="41.656" size="0.889" layer="27" ratio="11" rot="R270"/>
 </element>
 <element name="R2" library="Seeed-OPL-Resistor" package="R0805" value="82K" x="30.988" y="3.556" smashed="yes" rot="R180">
@@
 <via x="4.826" y="9.779" extent="1-16" drill="0.4318"/>
 <wire x1="6.35" y1="9.779" x2="4.826" y2="9.779" width="0.4064" layer="1"/>
-<wire x1="30.734" y1="41.275" x2="30.734" y2="42.795" width="0.508" layer="1"/>
-<wire x1="30.734" y1="42.795" x2="32.655" y2="44.716" width="0.508" layer="1"/>
+<wire x1="30.734" y1="41.021" x2="30.734" y2="42.922" width="0.508" layer="1"/>
+<wire x1="30.734" y1="42.922" x2="32.655" y2="44.843" width="0.508" layer="1"/>
 <wire x1="69.723" y1="38.862" x2="68.453" y2="38.862" width="0.254" layer="1"/>
 <wire x1="68.453" y1="38.862" x2="68.199" y2="39.116" width="0.254" layer="1"/>
@@
 <contactref element="X1" pad="TIP"/>
 <contactref element="F1" pad="1"/>
-<wire x1="34.655" y1="44.716" x2="34.655" y2="40.91" width="0.508" layer="1"/>
-<wire x1="34.655" y1="40.91" x2="34.671" y2="40.767" width="0.508" layer="1"/>
+<wire x1="34.655" y1="44.843" x2="34.655" y2="40.656" width="0.508" layer="1"/>
+<wire x1="34.655" y1="40.656" x2="34.671" y2="40.513" width="0.508" layer="1"/>
 <wire x1="44.423" y1="36.43" x2="41.383" y2="36.43" width="0.508" layer="1"/>
 <wire x1="41.383" y1="36.43" x2="40.005" y2="35.052" width="0.508" layer="1"/>
 <wire x1="40.005" y1="35.052" x2="37.211" y2="35.052" width="0.508" layer="1"/>
 <wire x1="37.211" y1="35.052" x2="36.322" y2="35.941" width="0.508" layer="1"/>
-<wire x1="36.322" y1="35.941" x2="36.322" y2="40.513" width="0.508" layer="1"/>
-<wire x1="36.322" y1="40.513" x2="36.068" y2="40.767" width="0.508" layer="1"/>
-<wire x1="36.068" y1="40.767" x2="34.671" y2="40.767" width="0.508" layer="1"/>
+<wire x1="36.322" y1="35.941" x2="36.322" y2="40.259" width="0.508" layer="1"/>
+<wire x1="36.322" y1="40.259" x2="36.068" y2="40.513" width="0.508" layer="1"/>
+<wire x1="36.068" y1="40.513" x2="34.671" y2="40.513" width="0.508" layer="1"/>
 </signal>
 <signal name="N$18">
@@
 <contactref element="F1" pad="2"/>
 <contactref element="SW1" pad="3"/>
-<wire x1="34.671" y1="37.973" x2="30.734" y2="37.973" width="0.508" layer="1"/>
+<wire x1="34.671" y1="37.719" x2="30.734" y2="37.719" width="0.508" layer="1"/>
 <wire x1="22.507" y1="42.855" x2="26.487" y2="42.855" width="0.508" layer="1"/>
 <wire x1="26.487" y1="42.855" x2="27.559" y2="41.783" width="0.508" layer="1"/>
-<wire x1="27.559" y1="41.783" x2="27.559" y2="38.862" width="0.508" layer="1"/>
-<wire x1="27.559" y1="38.862" x2="28.448" y2="37.973" width="0.508" layer="1"/>
-<wire x1="28.448" y1="37.973" x2="30.734" y2="37.973" width="0.508" layer="1"/>
+<wire x1="27.559" y1="41.783" x2="27.559" y2="38.608" width="0.508" layer="1"/>
+<wire x1="27.559" y1="38.608" x2="28.448" y2="37.719" width="0.508" layer="1"/>
+<wire x1="28.448" y1="37.719" x2="30.734" y2="37.719" width="0.508" layer="1"/>
 </signal>
 <signal name="N$19">
